File: hardware/ursp-pll-board/Versie 5.brd (EAGLE design)
At the start: 108 x 84 mm, 96 parts, among them IC1 MAX2870ETJ+T, IC2 LMK1C1103PWR, IC3 LMK1C1103PWR, IC4 LP5912-3.0DRVR, IC6 REF35180QDBVR, IC7 SN74AUP1T58DRYR, J1 60312202111527, J2 60312202111527, J3 60312202111527, J6 60312202111527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

Commit message: Changed values of loop filter
Parts:
- C23: value 100n -> 10u
- R6: value 240 -> 1k
- R7: value 30.1 -> 100
- R8: value 91 -> 330
Changed lines of the file:
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@@
 <attribute name="VALUE" x="24.955" y="38.125" size="1.27" layer="27" rot="R90"/>
 </element>
-<element name="C23" library="rcl" package="C0603" value="100n" x="21.12" y="35.135" smashed="yes" rot="R90">
+<element name="C23" library="rcl" package="C0603" value="10u" x="21.12" y="35.135" smashed="yes" rot="R90">
 <attribute name="NAME" x="36.3275" y="38.9625" size="0.8128" layer="25" font="vector" ratio="14" rot="R90"/>
 <attribute name="VALUE" x="23.025" y="34.5" size="1.27" layer="27" rot="R90"/>
@@
 <attribute name="VALUE" x="10.04" y="38.97" size="1.27" layer="27" rot="R270"/>
 </element>
-<element name="R6" library="rcl" package="R0603" value="240" x="23.05" y="35.135" smashed="yes" rot="R270">
+<element name="R6" library="rcl" package="R0603" value="1k" x="23.05" y="35.135" smashed="yes" rot="R270">
 <attribute name="NAME" x="37.64" y="38.9625" size="0.8128" layer="25" font="vector" ratio="14" rot="R90"/>
 <attribute name="VALUE" x="21.145" y="35.77" size="1.27" layer="27" rot="R270"/>
 </element>
-<element name="R7" library="rcl" package="R0603" value="30.1" x="25" y="35.135" smashed="yes" rot="R90">
+<element name="R7" library="rcl" package="R0603" value="100" x="25" y="35.135" smashed="yes" rot="R90">
 <attribute name="NAME" x="38.9475" y="38.9625" size="0.8128" layer="25" font="vector" ratio="14" rot="R90"/>
 <attribute name="VALUE" x="26.905" y="34.5" size="1.27" layer="27" rot="R90"/>
 </element>
-<element name="R8" library="rcl" package="R0603" value="91" x="23.05" y="31.425" smashed="yes" rot="R90">
+<element name="R8" library="rcl" package="R0603" value="330" x="23.05" y="31.425" smashed="yes" rot="R90">
 <attribute name="NAME" x="25.635" y="24.4525" size="0.8128" layer="25" font="vector" ratio="14" rot="R270"/>
 <attribute name="VALUE" x="24.955" y="30.79" size="1.27" layer="27" rot="R90"/>
